File: Kicad/ide-ram-a500.sch (KiCad schematic (older format))
At the start: 27 parts, among them J1 power, J2 LED, J3 LED2, J4 INT2OVR, J5 INT2, J6 JTAG, J7 IDE, U1 68000D socket, U2 XC95144XL-TQ100, U3 SPX3819M5-L-3-3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

Commit message: Updated CPLD code with new autoconfig, new ranger-maprom, rewritten IDE ; new MapROM software ; 0.2 hardware
Parts:
- added U13: XC6206PxxxMR, Package_TO_SOT_SMD:SOT-23, symbol Regulator_Linear:XC6206PxxxMR
Connections:
- net +3V3: now also U13.2 (VO)
- net +5V: now also U13.3 (VI)
- net GND: now also U13.1 (GND)
Other:
- note added: "Changelog :\nv0.2 :\nAdd XC6206 footprint"
- note added: "alternative footprint"
- moved on the sheet: C2, C6, U3
Changed lines of the file:
@@
 Title "IDE RAM A500"
 Date "2020-05-07"
-Rev "0.1"
+Rev "0.2"
 Comp "FLACO 2020 - Unknown licence, see projects below"
 Comment1 "Inspired by original design and code of ide68k v425 by Mika Leinonen"
@@
 L Regulator_Linear:SPX3819M5-L-3-3 U3
 U 1 1 5E93BE54
-P 14050 7250
-F 0 "U3" H 14050 7592 50  0000 C CNN
-F 1 "SPX3819M5-L-3-3" H 14050 7501 50  0000 C CNN
-F 2 "Package_TO_SOT_SMD:SOT-23-5" H 14050 7575 50  0001 C CNN
-F 3 "https://www.exar.com/content/document.ashx?id=22106&languageid=1033&type=Datasheet&partnumber=SPX3819&filename=SPX3819.pdf&part=SPX3819" H 14050 7250 50  0001 C CNN
-	1    14050 7250
+P 13600 7250
+F 0 "U3" H 13600 7592 50  0000 C CNN
+F 1 "SPX3819M5-L-3-3" H 13600 7501 50  0000 C CNN
+F 2 "Package_TO_SOT_SMD:SOT-23-5" H 13600 7575 50  0001 C CNN
+F 3 "https://www.exar.com/content/document.ashx?id=22106&languageid=1033&type=Datasheet&partnumber=SPX3819&filename=SPX3819.pdf&part=SPX3819" H 13600 7250 50  0001 C CNN
+	1    13600 7250
 	1    0    0    -1
 $EndComp
@@
 L power:+5V #PWR013
 U 1 1 5E962832
-P 13250 7150
-F 0 "#PWR013" H 13250 7000 50  0001 C CNN
-F 1 "+5V" H 13265 7323 50  0000 C CNN
-F 2 "" H 13250 7150 50  0001 C CNN
-F 3 "" H 13250 7150 50  0001 C CNN
-	1    13250 7150
+P 12800 7150
+F 0 "#PWR013" H 12800 7000 50  0001 C CNN
+F 1 "+5V" H 12815 7323 50  0000 C CNN
+F 2 "" H 12800 7150 50  0001 C CNN
+F 3 "" H 12800 7150 50  0001 C CNN
+	1    12800 7150
 	1    0    0    -1
 $EndComp
@@
 L power:+3.3V #PWR028
 U 1 1 5E962E41
-P 14900 7150
-F 0 "#PWR028" H 14900 7000 50  0001 C CNN
-F 1 "+3.3V" H 14915 7323 50  0000 C CNN
-F 2 "" H 14900 7150 50  0001 C CNN
-F 3 "" H 14900 7150 50  0001 C CNN
-	1    14900 7150
+P 14450 7150
+F 0 "#PWR028" H 14450 7000 50  0001 C CNN
+F 1 "+3.3V" H 14465 7323 50  0000 C CNN
+F 2 "" H 14450 7150 50  0001 C CNN
+F 3 "" H 14450 7150 50  0001 C CNN
+	1    14450 7150
 	1    0    0    -1
 $EndComp
@@
 L Device:C_Small C2
 U 1 1 5E963578
-P 13400 7250
-F 0 "C2" H 13492 7296 50  0000 L CNN
-F 1 "10u" H 13492 7205 50  0000 L CNN
-F 2 "Capacitor_SMD:C_0805_2012Metric" H 13400 7250 50  0001 C CNN
-F 3 "~" H 13400 7250 50  0001 C CNN
-	1    13400 7250
-	1    0    0    -1
-$EndComp
-Wire Wire Line
-	13750 7150 13400 7150
-Connection ~ 13400 7150
-Wire Wire Line
-	13400 7150 13250 7150
-Wire Wire Line
-	13750 7250 13750 7150
-Connection ~ 13750 7150
-Wire Wire Line
-	14350 7150 14550 7150
-Wire Wire Line
-	13400 7350 13400 7550
-Wire Wire Line
-	13250 7550 13400 7550
+P 12950 7250
+F 0 "C2" H 13042 7296 50  0000 L CNN
+F 1 "10u" H 13042 7205 50  0000 L CNN
+F 2 "Capacitor_SMD:C_0805_2012Metric" H 12950 7250 50  0001 C CNN
+F 3 "~" H 12950 7250 50  0001 C CNN
+	1    12950 7250
+	1    0    0    -1
+$EndComp
+Wire Wire Line
+	13300 7150 12950 7150
+Connection ~ 12950 7150
+Wire Wire Line
+	12950 7150 12800 7150
+Wire Wire Line
+	13300 7250 13300 7150
+Connection ~ 13300 7150
+Wire Wire Line
+	13900 7150 14100 7150
+Wire Wire Line
+	12950 7350 12950 7550
+Wire Wire Line
+	12800 7550 12950 7550
 $Comp
 L Device:C_Small C6
 U 1 1 5E96573B
-P 14550 7250
-F 0 "C6" H 14642 7296 50  0000 L CNN
-F 1 "10u" H 14642 7205 50  0000 L CNN
-F 2 "Capacitor_SMD:C_0805_2012Metric" H 14550 7250 50  0001 C CNN
-F 3 "~" H 14550 7250 50  0001 C CNN
-	1    14550 7250
-	1    0    0    -1
-$EndComp
-Connection ~ 14550 7150
-Wire Wire Line
-	14550 7150 14900 7150
-Wire Wire Line
-	14550 7350 14550 7550
-Wire Wire Line
-	14550 7550 14050 7550
-Connection ~ 14050 7550
+P 14100 7250
+F 0 "C6" H 14192 7296 50  0000 L CNN
+F 1 "10u" H 14192 7205 50  0000 L CNN
+F 2 "Capacitor_SMD:C_0805_2012Metric" H 14100 7250 50  0001 C CNN
+F 3 "~" H 14100 7250 50  0001 C CNN
+	1    14100 7250
+	1    0    0    -1
+$EndComp
+Connection ~ 14100 7150
+Wire Wire Line
+	14100 7150 14450 7150
+Wire Wire Line
+	14100 7350 14100 7550
+Wire Wire Line
+	14100 7550 13600 7550
+Connection ~ 13600 7550
 $Comp
 L power:GND #PWR014
 U 1 1 5E9664A6
-P 13250 7550
-F 0 "#PWR014" H 13250 7300 50  0001 C CNN
-F 1 "GND" H 13255 7377 50  0000 C CNN
-F 2 "" H 13250 7550 50  0001 C CNN
-F 3 "" H 13250 7550 50  0001 C CNN
-	1    13250 7550
-	1    0    0    -1
-$EndComp
-Connection ~ 13400 7550
-Wire Wire Line
-	13400 7550 14050 7550
+P 12800 7550
+F 0 "#PWR014" H 12800 7300 50  0001 C CNN
+F 1 "GND" H 12805 7377 50  0000 C CNN
+F 2 "" H 12800 7550 50  0001 C CNN
+F 3 "" H 12800 7550 50  0001 C CNN
+	1    12800 7550
+	1    0    0    -1
+$EndComp
+Connection ~ 12950 7550
+Wire Wire Line
+	12950 7550 13600 7550
 $Comp
 L power:+3.3V #PWR04
@@
 Wire Wire Line
 	10850 8100 10850 8350
-NoConn ~ 14350 7250
+NoConn ~ 13900 7250
 NoConn ~ 7800 3950
 $Comp
@@
 Text Notes 13200 5900 0    50   ~ 0
 PCB ready for CY62177ESL\nhowever due to the price of this chip only CY62167ELL are tested.\nStay away from low voltage versions of this chip.
+Text Notes 800  10900 0    50   ~ 0
+Changelog :\nv0.2 :\nAdd XC6206 footprint
+$Comp
+L Regulator_Linear:XC6206PxxxMR U13
+U 1 1 5FC2F377
+P 15200 7150
+F 0 "U13" H 15200 7392 50  0000 C CNN
+F 1 "XC6206PxxxMR" H 15200 7301 50  0000 C CNN
+F 2 "Package_TO_SOT_SMD:SOT-23" H 15200 7375 50  0001 C CIN
+F 3 "https://www.torexsemi.com/file/xc6206/XC6206.pdf" H 15200 7150 50  0001 C CNN
+	1    15200 7150
+	1    0    0    -1
+$EndComp
+$Comp
+L power:+3.3V #PWR0103
+U 1 1 5FC34A57
+P 15650 7150
+F 0 "#PWR0103" H 15650 7000 50  0001 C CNN
+F 1 "+3.3V" H 15665 7323 50  0000 C CNN
+F 2 "" H 15650 7150 50  0001 C CNN
+F 3 "" H 15650 7150 50  0001 C CNN
+	1    15650 7150
+	1    0    0    -1
+$EndComp
+$Comp
+L power:+5V #PWR0104
+U 1 1 5FC3521A
+P 14750 7150
+F 0 "#PWR0104" H 14750 7000 50  0001 C CNN
+F 1 "+5V" H 14765 7323 50  0000 C CNN
+F 2 "" H 14750 7150 50  0001 C CNN
+F 3 "" H 14750 7150 50  0001 C CNN
+	1    14750 7150
+	1    0    0    -1
+$EndComp
+$Comp
+L power:GND #PWR0105
+U 1 1 5FC3586B
+P 15200 7450
+F 0 "#PWR0105" H 15200 7200 50  0001 C CNN
+F 1 "GND" H 15205 7277 50  0000 C CNN
+F 2 "" H 15200 7450 50  0001 C CNN
+F 3 "" H 15200 7450 50  0001 C CNN
+	1    15200 7450
+	1    0    0    -1
+$EndComp
+Wire Wire Line
+	14900 7150 14750 7150
+Wire Wire Line
+	15500 7150 15650 7150
+Text Notes 14850 6750 0    50   ~ 0
+alternative footprint
 $EndSCHEMATC
