File: Kicad/a500-ide-ram.kicad_sch (KiCad schematic)
At the start: 28 parts, among them J1 power, J2 LED, J3 LED2, J4 INT2OVR, J5 INT2, J6 JTAG, J7 IDE, U1 68000D socket, U13 XC6206PxxxMR, U2 XC95144XL-TQ100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

Commit message: KiCAD : correct license on schematic and PCB
Parts:
- added FID1: Fiducial, Sassa:CC_BY_NC_SA_square_silkscreen, symbol Mechanical:Fiducial
- gave numbers to parts that had none: 1
Other:
- company: FLACO 2020 - Unknown licence, see projects below -> FLACO 2020 CC-BY-NC-SA
Changed lines of the file:
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@@
     (date "2020-05-07")
     (rev "0.2")
-    (company "FLACO 2020 - Unknown licence, see projects below")
+    (company "FLACO 2020 CC-BY-NC-SA")
     (comment 1 "Inspired by original design and code of ide68k v425 by Mika Leinonen")
     (comment 2 "http://www.mkl211015.altervista.org/ide/ide68k.html")
@@
   (symbol (lib_id "power:+3.3V") (at 367.03 181.61 0) (unit 1)
     (in_bom yes) (on_board yes)
-    (property "Reference" "" (id 0) (at 367.03 185.42 0)
+    (property "Reference" "#PWR028" (id 0) (at 367.03 185.42 0)
       (effects (font (size 1.27 1.27)) hide)
     )
@@
   (symbol (lib_id "power:+3.3V") (at 102.87 35.56 0) (unit 1)
     (in_bom yes) (on_board yes)
-    (property "Reference" "" (id 0) (at 102.87 39.37 0)
+    (property "Reference" "#PWR04" (id 0) (at 102.87 39.37 0)
       (effects (font (size 1.27 1.27)) hide)
     )
@@
   (symbol (lib_id "power:PWR_FLAG") (at 199.39 165.1 90) (unit 1)
     (in_bom yes) (on_board yes)
-    (property "Reference" "" (id 0) (at 197.485 165.1 0)
+    (property "Reference" "#FLG0101" (id 0) (at 197.485 165.1 0)
       (effects (font (size 1.27 1.27)) hide)
     )
@@
   (symbol (lib_id "power:PWR_FLAG") (at 201.93 43.18 270) (unit 1)
     (in_bom yes) (on_board yes)
-    (property "Reference" "" (id 0) (at 203.835 43.18 0)
+    (property "Reference" "#FLG0102" (id 0) (at 203.835 43.18 0)
       (effects (font (size 1.27 1.27)) hide)
     )
@@
   (symbol (lib_id "power:+3.3V") (at 232.41 212.09 0) (unit 1)
     (in_bom yes) (on_board yes)
-    (property "Reference" "" (id 0) (at 232.41 215.9 0)
+    (property "Reference" "#PWR0101" (id 0) (at 232.41 215.9 0)
       (effects (font (size 1.27 1.27)) hide)
     )
@@
   (symbol (lib_id "Device:R_Small") (at 77.47 207.01 0) (unit 1)
     (in_bom yes) (on_board yes)
-    (property "Reference" "" (id 0) (at 78.9686 205.8416 0)
+    (property "Reference" "RLED1" (id 0) (at 78.9686 205.8416 0)
       (effects (font (size 1.27 1.27)) (justify left))
     )
@@
   (symbol (lib_id "power:+3.3V") (at 77.47 204.47 0) (unit 1)
     (in_bom yes) (on_board yes)
-    (property "Reference" "" (id 0) (at 77.47 208.28 0)
+    (property "Reference" "#PWR03" (id 0) (at 77.47 208.28 0)
       (effects (font (size 1.27 1.27)) hide)
     )
@@
   (symbol (lib_id "power:+3.3V") (at 154.94 179.07 0) (unit 1)
     (in_bom yes) (on_board yes)
-    (property "Reference" "" (id 0) (at 154.94 182.88 0)
+    (property "Reference" "#PWR06" (id 0) (at 154.94 182.88 0)
       (effects (font (size 1.27 1.27)) hide)
     )
@@
   (symbol (lib_id "power:+3.3V") (at 332.74 208.28 0) (unit 1)
     (in_bom yes) (on_board yes)
-    (property "Reference" "" (id 0) (at 332.74 212.09 0)
+    (property "Reference" "#PWR011" (id 0) (at 332.74 212.09 0)
       (effects (font (size 1.27 1.27)) hide)
     )
@@
   (symbol (lib_id "power:+3.3V") (at 397.51 181.61 0) (unit 1)
     (in_bom yes) (on_board yes)
-    (property "Reference" "" (id 0) (at 397.51 185.42 0)
+    (property "Reference" "#PWR0103" (id 0) (at 397.51 185.42 0)
       (effects (font (size 1.27 1.27)) hide)
     )
@@
     )
     (pin "1")
+  )
+  (symbol (lib_id "Mechanical:Fiducial") (at 393.7 245.11 0) (unit 1)
+    (in_bom yes) (on_board yes) (fields_autoplaced)
+    (property "Reference" "FID1" (id 0) (at 396.24 243.8399 0)
+      (effects (font (size 1.27 1.27)) (justify left))
+    )
+    (property "Value" "Fiducial" (id 1) (at 396.24 246.3799 0)
+      (effects (font (size 1.27 1.27)) (justify left))
+    )
+    (property "Footprint" "Sassa:CC_BY_NC_SA_square_silkscreen" (id 2) (at 393.7 245.11 0)
+      (effects (font (size 1.27 1.27)) hide)
+    )
+    (property "Datasheet" "~" (id 3) (at 393.7 245.11 0)
+      (effects (font (size 1.27 1.27)) hide)
+    )
   )
   (sheet_instances
@@
       (reference "D1") (unit 1) (value "BAT54A") (footprint "Package_TO_SOT_SMD:SOT-23")
     )
+    (path "/7d989f0b-29a3-4e20-8f77-f4a88c057624"
+      (reference "FID1") (unit 1) (value "Fiducial") (footprint "Sassa:CC_BY_NC_SA_square_silkscreen")
+    )
     (path "/00000000-0000-0000-0000-00005eb8a8aa"
